File: Board/BreadBoardPowerSupply.kicad_pcb (KiCad board)
At the start: 2 copper layers, 6 parts, among them CON1 BARREL_JACK, U1 7805

Commit message: Update schematics (added polarised capacitors)
Parts:
- C1, C2: value C -> CP
Changed lines of the file:
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@@
     (links 11)
     (no_connects 0)
-    (area 120.210476 83.51 164.134286 110.74)
+    (area 0 0 0 0)
     (thickness 1.6)
     (drawings 0)
@@
       (effects (font (size 1 1) (thickness 0.15)) (justify mirror))
     )
-    (fp_text value C (at 2.5 -6.3 270) (layer B.Fab)
+    (fp_text value CP (at 2.5 -6.3 270) (layer B.Fab)
       (effects (font (size 1 1) (thickness 0.15)) (justify mirror))
     )
@@
       (effects (font (size 1 1) (thickness 0.15)) (justify mirror))
     )
-    (fp_text value C (at 1.25 -3.8 180) (layer B.Fab)
+    (fp_text value CP (at 1.25 -3.8 180) (layer B.Fab)
       (effects (font (size 1 1) (thickness 0.15)) (justify mirror))
     )
